File: main-board.brd (EAGLE design)
At the start: 171.1 x 156.7 mm, 61 parts, among them IC1 7805T, IC2 7805T, IC3 7805T, J5 XT-60BATT_LABEL, J6 43045-0613, J7 43045-0613, J8 43045-0613, J9 43045-0613, X1 22-23-2021, X2 5566-4, X3 5566-4, X4 5566-4, X5 5566-4

Commit message: removed redundant files
Parts:
- removed J9: 43045-0613, 43045-0613:43045-0613
- removed JP5, JP6: (no value), pinhead:2X15
- removed LED1, LED2, LED3, LED4, LED5: (no value), led:1206
- removed R5: (no value), resistor:R1206
- removed S2, S3: TME1, switch-misc:TME1
- removed SV1, SV2, SV3, SV4: (no value), con-lsta:FE10
- removed SV13, SV18, SV6, SV7: (no value), con-lsta:FE08
- removed SV14: (no value), con-lstb:MA10-1
- removed SV17: (no value), con-lstb:MA08-1
- removed U$4: BUCK, BUCK:BUCK
- removed U$5: (no value), switch_DA10:DA10
- removed U2, U3: (no value), LP38690DT-3.3:TO228P1042X238-3N
- removed X5: 5566-4, con-molex:5566-4
- added 3V3_LD, 5V_LD, NRF_STATUS: (no value), led:CHIPLED_1206
- added C11, C12, C15: 0.1uF, rcl:C1206
- added C13, C14, C16: 4.7uF, rcl:C1206
- added IC4: AM26LS32ACPWR, SamacSys_Parts:SOP65P640X120-16N
- added J10: XT60-M, XT60-M:AMASS_XT60-M
- added M1: WIRELESS-NRF24L01-PA-EXT, diy_modules_2:WIRELESS-NRD24L01-PA-EXT
- added MD1, MD2, MD3, MD4, MD5: KRSSG_MOTOR_DRIVER, KRSSG_MOTOR_DRIVER:KRSSG_MOTOR_DRIVER
- added S1: DTS-6, switch-tact:DTS-6
- C1, C10, C2, C3, C4, C5, C6, C9: value 47uF -> 0.1uF
- C7, C8: value 47uF -> 4.7uF
- IC1: value 7805T -> 7805DT; device linear:TO220H -> linear:TO252
- IC2: value 7805T -> AP7365-33ERG-13; device linear:TO220H -> SamacSys_Parts:SOT230P700X180-4N
- IC3: value 7805T -> AM26LS32ACPWR; device linear:TO220H -> SamacSys_Parts:SOP65P640X120-16N
- J2, J4: value (none) -> 43045-0613; device SparkFun-Connectors:2X5-SHROUDED_LOCK -> 43045-0613:43045-0613
- J5: value XT-60BATT_LABEL -> (none); device RoboJackets-Connectors:XT-60 -> SparkFun-Connectors:2X5-SHROUDED_LOCK
- J8: value 43045-0613 -> (none); device 43045-0613:43045-0613 -> SparkFun-Connectors:2X5-SHROUDED_LOCK
- JP1: device pinhead:2X20 -> pinhead:1X03
- JP2: device pinhead:2X20 -> pinhead:1X06
- R1: value (none) -> 10K; device resistor:R1206 -> rcl:M1206
- R2, R3, R4: value (none) -> 1K; device resistor:R1206 -> rcl:M1206
- SV5: device con-lstb:MA08-1 -> pinhead:1X08
- SV8: device con-lsta:FE08 -> pinhead:1X08
- U1: value (none) -> STM32F103VCT6; device LP38690DT-3.3:TO228P1042X238-3N -> STM32F103VCT6:LQFP100-14X14MM
- X1: value 22-23-2021 -> 5566-4; device con-molex:22-23-2021 -> con-molex:5566-4
- moved IC3 313.4 mm to (-35.6, -238.8), flipped to the top, turned to 0 degrees
- moved IC2 305.2 mm to (-53.3, -231.1), flipped to the top
- moved SV8 301.9 mm to (-85.1, -246.4), turned to 0 degrees
- moved C1 297.0 mm to (-41.9, -231.1), flipped to the top
- moved C3 295.3 mm to (-29.2, -231.1), flipped to the top, turned to 0 degrees
- moved C4 295.0 mm to (-22.9, -231.1), flipped to the top
- moved C5 290.6 mm to (-16.5, -231.1), flipped to the top, turned to 0 degrees
- moved IC1 287.9 mm to (-33.0, -215.9), flipped to the top
- moved C9 287.1 mm to (8.89, -231.1), flipped to the top, turned to 0 degrees
- moved R1 273.5 mm to (-62.2, -238.8), flipped to the top, turned to 0 degrees
- moved R4 268.6 mm to (-47.0, -238.8), flipped to the top, turned to 0 degrees
- moved R2 266.7 mm to (-57.1, -238.8), flipped to the top, turned to 0 degrees
- moved R3 266.4 mm to (-52.1, -238.8), flipped to the top, turned to 0 degrees
- moved X4 265.5 mm to (-69.8, -219.7), flipped to the top, turned to 0 degrees
- moved J5 261.8 mm to (-81.3, -199.4), flipped to the top, turned to 0 degrees
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Connections:
- removed net 12V: C1.1, C4.1, C9.1, IC1.1, IC2.1, IC3.1, R4.1, SV14.10, SV14.9, U$4.VOUT
- removed net 5V1: C5.1, IC2.3, R1.1, X1.2
- removed net 5V_ESP: C10.1, IC3.3, JP6.1, JP6.2
- removed net ESP_EN: JP2.24
- removed net ESP_REC: JP6.15, JP6.16
- removed net ESP_RX: JP1.26, JP5.23, JP5.24, S2.1, S2.5
- removed net ESP_TRANS: JP6.13, JP6.14
- removed net ESP_TX: JP1.28, JP5.25, JP5.26, S3.1, S3.5
- removed net FPGA_REC: JP2.26, R5.1
- removed net INPUT: U$5.P$1, U1.1, U1.3, U2.1, U2.3, U3.1, U3.3
- removed net N$10: LED3.A, R3.2
- removed net N$11: JP5.11, JP5.12
- removed net N$12: JP5.13, JP5.14
- removed net N$13: LED4.A, R4.2
- removed net N$14: JP5.15, JP5.16
- removed net N$15: JP5.17, JP5.18
- removed net N$16: LED5.A, R5.2
- removed net N$17: JP5.19, JP5.20
- removed net N$18: JP5.21, JP5.22
- removed net N$23: JP5.27, JP5.28
- removed net N$24: JP5.29, JP5.30
- removed net N$27: JP6.5, JP6.6
- removed net N$28: JP6.7, JP6.8
- removed net N$29: JP6.10, JP6.9
- removed net N$30: JP6.11, JP6.12
- removed net N$38: JP6.27, JP6.28
- removed net N$39: JP6.29, JP6.30
- removed net N$41: JP6.25, JP6.26
- removed net N$6: JP5.5, JP5.6
- removed net N$8: JP5.7, JP5.8
- removed net N$9: JP5.10, JP5.9
- removed net SUPP: J5.BATT, U$5.P$2
- new net 5V_EXT: JP1.3
- new net 5V_REG: C13.1, IC2.2, IC2.4, IC3.16, IC3.4, IC4.16, IC4.4, J1.2, J2.5, J3.2, J4.5, J5.2, J6.5, J7.5, J8.2, JP1.2, MD1.5V, MD2.5V, MD3.5V, MD4.5V, MD5.5V, R2.2, SV8.5
- new net M1EAN: IC3.2, J1.5
- new net M1EA_RECT: IC3.3
- new net M1EBN: IC3.7, J1.7
- new net M1EB_RECT: IC3.5
- new net M2EAN: J3.5
- new net M2EA_RECT: IC3.13
- new net M2EBN: IC3.9, J3.7
- new net M2EB_RECT: IC3.11
- new net M3EAN: IC3.15, IC4.2, J5.5
- new net M3EA_RECT: IC4.3
- new net M3EBN: IC4.7, J5.7
- new net M3EB_RECT: IC4.5
- new net M4EAN: IC4.15, J8.5
- new net M4EA_RECT: IC4.13
- new net M4EBN: IC4.9, J8.7
- new net M4EB_RECT: IC4.11
- new net N$2: 3V3_LD.A, R3.1
- new net N$3: C11.1, IC1.2, JP1.1
- new net NRF_CE: M1.3
- new net NRF_CSN: M1.4, NRF_STATUS.C
- new net NRF_IRQ: M1.8
- new net NRF_MISO: M1.7
- new net NRF_MOSI: M1.6
- new net NRF_SCK: M1.5
- new net NRST: C10.1, JP2.5, S1.1, S1.2
- new net SWCLK: JP2.2, U1.76
- new net SWDIO: JP2.4, U1.72
- new net SWO: JP2.6, U1.89
- net 18V: now also C12.1, IC1.1, MD1.18V, MD1.18V_2, MD2.18V, MD2.18V_2, MD3.18V, MD3.18V_2, MD4.18V, MD4.18V_2, MD5.18V, MD5.18V_2; no longer R3.1, SV1.10, SV1.9, SV2.10, SV2.9, SV3.10, SV3.9, SV4.10, SV4.9, U$4.VIN, U1.2, U2.2, U3.2
- net CHARGE: no longer JP2.16
- net DONE: no longer JP2.18
- net GND: now also 3V3_LD.C, 5V_LD.C, C11.2, C12.2, C13.2, C14.2, C15.2, C16.2, C2.2, C6.2, C7.2, C8.2, IC1.3, IC2.1, IC3.12, IC3.8, IC4.12, IC4.8, J2.4, J4.4, J5.3, J8.3, JP2.3, M1.1, MD1.GND, MD1.GND_2, MD2.GND, MD2.GND_2, MD3.GND, MD3.GND_2, MD4.GND, MD4.GND_2, MD5.GND, MD5.GND_2, R1.1, S1.3, S1.4, U1.10, U1.19, U1.20, U1.27, U1.49, U1.74, U1.99; no longer C2.1, C6.1, C7.1, C8.1, IC1.2, IC2.2, IC3.2, J2.3, J4.3, J5.GND, J8.4, J9.4, JP1.1, JP1.19, JP1.20, JP1.39, JP2.2, JP2.40, JP5.3, JP5.4, JP6.3, JP6.4, LED1.C, LED2.C, LED3.C, LED4.C, LED5.C, S2.2, S2.4, S3.2, S3.4, SV1.1, SV1.2, SV14.1, SV14.2, SV2.1, SV2.2, SV3.1, SV3.2, SV4.1, SV4.2, U$4.GND, U$4.GNDO, X1.1
- net IR1: no longer JP2.25
- net IR2: no longer JP2.27
- net IR3: no longer JP2.15
- net KICK: no longer JP2.22
- net KICK_CHIP: no longer JP2.20
- net M11: now also MD1.M1, MD1.M1_2; no longer SV6.6, SV6.7
- net M11A: now also MD1.M1A; no longer JP1.13, SV2.8
- net M11B: now also MD1.M1B; no longer JP1.11, SV2.7
- net M12: now also MD1.M2, MD1.M2_2; no longer SV6.4, SV6.5
- net M12A: now also MD1.M2A; no longer JP1.9, SV2.6
- net M12B: now also MD1.M2B; no longer JP1.7, SV2.5
- net M13: now also MD1.M3, MD1.M3_2; no longer SV6.2, SV6.3
- net M13A: now also MD1.M3A; no longer JP1.5, SV2.4
- net M13B: now also MD1.M3B; no longer JP1.3, SV2.3
- net M1ACS_OUT: now also MD1.MACS_OUT; no longer C2.2, JP6.17, JP6.18, SV6.8
- net M1EA: now also IC3.1; no longer JP1.6
- net M1EB: now also IC3.6; no longer JP1.4
- net M1H1: no longer JP1.8
- net M1H2: no longer JP1.10
- net M1H3: no longer JP1.12
- net M21: now also MD2.M1, MD2.M1_2, X1.1; no longer SV7.6, SV7.7, X2.1
- net M21A: now also MD2.M1A; no longer JP1.27, SV1.8
- net M21B: now also MD2.M1B; no longer JP1.29, SV1.7
- net M22: now also MD2.M2, MD2.M2_2, X1.2; no longer SV7.4, SV7.5, X2.2
- net M22A: now also MD2.M2A; no longer JP1.31, SV1.6
- net M22B: now also MD2.M2B; no longer JP1.33, SV1.5
- net M23: now also MD2.M3, MD2.M3_2, X1.3; no longer SV7.2, SV7.3, X2.3
- net M23A: now also MD2.M3A; no longer JP1.35, SV1.4
- net M23B: now also MD2.M3B; no longer JP1.37, SV1.3
- net M2ACS_OUT: now also MD2.MACS_OUT; no longer C6.2, JP6.19, JP6.20, SV7.8
- net M2EA: no longer JP1.32
- net M2EB: now also IC3.10; no longer JP1.30
- net M2H1: now also J2.1; no longer J7.1, JP1.34
- net M2H2: now also J2.2; no longer J7.2, JP1.36
- net M2H3: now also J2.3; no longer J7.3, JP1.38
- net M31: now also MD3.M1, MD3.M1_2, X2.1; no longer SV13.6, SV13.7, X4.1
- net M31A: now also MD3.M1A; no longer JP2.4, SV3.8
- net M31B: now also MD3.M1B; no longer JP2.6, SV3.7
- net M32: now also MD3.M2, MD3.M2_2, X2.2; no longer SV13.4, SV13.5, X4.2
- net M32A: now also MD3.M2A; no longer JP2.8, SV3.6
- net M32B: now also MD3.M2B; no longer JP2.10, SV3.5
- net M33: now also MD3.M3, MD3.M3_2, X2.3; no longer SV13.2, SV13.3, X4.3
- net M33A: now also MD3.M3A; no longer JP2.12, SV3.4
- net M33B: now also MD3.M3B; no longer JP2.14, SV3.3
- net M3ACS_OUT: now also MD3.MACS_OUT; no longer C7.2, JP6.21, JP6.22, SV13.8
- net M3EA: now also IC3.14, IC4.1, J5.6; no longer J2.6, JP2.3
- net M3EB: now also IC4.6, J5.8; no longer J2.8, JP2.5
- net M3H1: now also J4.1; no longer J8.1, JP2.7
- net M3H2: now also J4.2; no longer J8.2, JP2.9
- net M3H3: now also J4.3; no longer J8.3, JP2.11
- net M41: now also MD4.M1, MD4.M1_2, X4.1; no longer SV18.6, SV18.7, X5.1
- net M41A: now also MD4.M1A; no longer JP2.38, SV4.8
- net M41B: now also MD4.M1B; no longer JP2.36, SV4.7
- net M42: now also MD4.M2, MD4.M2_2, X4.2; no longer SV18.4, SV18.5, X5.2
- net M42A: now also MD4.M2A; no longer JP2.34, SV4.6
- net M42B: now also MD4.M2B; no longer JP2.32, SV4.5
- net M43: now also MD4.M3, MD4.M3_2, X4.3; no longer SV18.2, SV18.3, X5.3
- net M43A: now also MD4.M3A; no longer JP2.30, SV4.4
- net M43B: now also MD4.M3B; no longer JP2.28, SV4.3
- net M4ACS_OUT: now also MD4.MACS_OUT; no longer C8.2, JP6.23, JP6.24, SV18.8
- net M4EA: now also IC4.14, J8.6; no longer J4.6, JP2.31
- net M4EB: now also IC4.10, J8.8; no longer J4.8, JP2.29
- net M4H1: now also J7.1; no longer J9.1, JP2.33
- net M4H2: now also J7.2; no longer J9.2, JP2.35
- net M4H3: now also J7.3; no longer J9.3, JP2.37
- net MD1: now also MD5.M1, MD5.M1_2; no longer SV17.6, SV17.7
- net MD1A: now also MD5.M1A; no longer JP1.15, SV14.8
- net MD1B: now also MD5.M1B; no longer JP1.17, SV14.7
- net MD2: now also MD5.M2, MD5.M2_2; no longer SV17.4, SV17.5
- net MD2A: now also MD5.M2A; no longer JP2.13, SV14.6
- net MD2B: now also MD5.M2B; no longer JP1.21, SV14.5
- net MD3: now also MD5.M3, MD5.M3_2; no longer SV17.2, SV17.3
- net MD3A: now also MD5.M3A; no longer JP1.23, SV14.4
- net MD3B: now also MD5.M3B; no longer JP1.25, SV14.3
- net MDACS_OUT: now also MD5.MACS_OUT; no longer SV17.8
- net MDH1: no longer JP1.16
- net MDH2: no longer JP1.18
- net MDH3: no longer JP2.17
- net N$1: now also R1.2, U1.94; no longer JP5.1, JP5.2
- net N$4: now also 5V_LD.A, R2.1; no longer LED1.A, R1.2
- net N$7: now also NRF_STATUS.A, R4.1; no longer LED2.A, R2.2
- net VCC: now also C1.1, C14.1, C15.1, C16.1, C2.1, C4.1, C5.1, C6.1, C7.1, C8.1, C9.1, IC2.3, JP2.1, M1.2, R3.2, R4.2, U1.100, U1.11, U1.21, U1.22, U1.28, U1.50, U1.6, U1.75; no longer IC1.3, J1.2, J2.2, J3.2, J4.2, J6.5, J7.5, J8.5, J9.5, R2.1, SV13.1, SV17.1, SV18.1, SV6.1, SV7.1, SV8.5
Routing:
- net VCC: track 478.6 -> 0.00 mm, vias 4 -> 0
- net 18V: track 406.7 -> 0.00 mm
- net GND: track 286.7 -> 0.00 mm, vias 2 -> 0
- net 12V: track 182.0 -> 0.00 mm, vias 1 -> 0
- net 5V1: track 158.6 -> 0.00 mm
- net M1ACS_OUT: track 130.7 -> 0.00 mm
- net IR3: track 103.1 -> 0.00 mm
- net M3ACS_OUT: track 90.7 -> 0.00 mm
- net 5V_ESP: track 88.1 -> 0.00 mm, vias 1 -> 0
- net KICK: track 87.6 -> 0.00 mm
- net KICK_CHIP: track 85.7 -> 0.00 mm
- net DONE: track 83.8 -> 0.00 mm
- net CHARGE: track 82.7 -> 0.00 mm, vias 1 -> 0
- net MDH1: track 76.7 -> 0.00 mm
- net MDH2: track 76.6 -> 0.00 mm
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