File: main-board.sch (EAGLE design)
At the start: 60 parts, among them IC1 7805T, IC2 7805T, IC3 7805T, J5 XT-60BATT_LABEL, J6 43045-0613, J7 43045-0613, J8 43045-0613, J9 43045-0613, X1 22-23-2021, X2 5566-4, X3 5566-4, X4 5566-4, X5 5566-4

Commit message: removed redundant files
Parts:
- removed J9: 43045-0613, 43045-0613:43045-0613
- removed JP5, JP6: (no value), pinhead:PINHD-2X15
- removed LED1, LED2, LED3, LED4, LED5: (no value), led:LEDSMT1206
- removed R5: (no value), resistor:R-EU_R1206
- removed S2, S3: TME1, switch-misc:TME1
- removed SV1, SV2, SV3, SV4: (no value), con-lsta:FE10-1
- removed SV13, SV18, SV6, SV7: (no value), con-lsta:FE08-1
- removed SV14: (no value), con-lstb:MA10-1
- removed SV17: (no value), con-lstb:MA08-1
- removed U$4: BUCK, BUCK:BUCK
- removed U$5: (no value), switch_DA10:SWITCH_DA10
- removed U2, U3: (no value), LP38690DT-3.3:LP38690DT-3.3
- removed X5: 5566-4, con-molex:5566-4
- added 3V3_LD, 5V_LD, NRF_STATUS: (no value), led:LEDCHIPLED_1206
- added C11, C12, C15: 0.1uF, rcl:C-USC1206
- added C13, C14, C16: 4.7uF, rcl:C-USC1206
- added IC4: AM26LS32ACPWR, SamacSys_Parts:AM26LS32ACPWR
- added J10: XT60-M, XT60-M:XT60-M
- added M1: WIRELESS-NRF24L01-PA-EXT, diy_modules_2:WIRELESS-NRF24L01-PA-EXT
- added MD1, MD2, MD3, MD4, MD5: KRSSG_MOTOR_DRIVER, KRSSG_MOTOR_DRIVER:KRSSG_MOTOR_DRIVER
- added S1: DTS-6, switch-tact:DTS-6
- C1, C10, C2, C3, C4, C5, C6, C9: value 47uF -> 0.1uF; device rcl:C-EUC1206 -> rcl:C-USC1206
- C7, C8: value 47uF -> 4.7uF; device rcl:C-EUC1206 -> rcl:C-USC1206
- IC1: value 7805T -> 7805DT; device linear:7805T -> linear:7805DT
- IC2: value 7805T -> AP7365-33ERG-13; device linear:7805T -> SamacSys_Parts:AP7365-33ERG-13
- IC3: value 7805T -> AM26LS32ACPWR; device linear:7805T -> SamacSys_Parts:AM26LS32ACPWR
- J2, J4: value (none) -> 43045-0613; device SparkFun-Connectors:CONN_05X2SHD_LOCK -> 43045-0613:43045-0613
- J5: value XT-60BATT_LABEL -> (none); device RoboJackets-Connectors:XT-60BATT_LABEL -> SparkFun-Connectors:CONN_05X2SHD_LOCK
- J8: value 43045-0613 -> (none); device 43045-0613:43045-0613 -> SparkFun-Connectors:CONN_05X2SHD_LOCK
- JP1: device pinhead:PINHD-2X20 -> pinhead:PINHD-1X3
- JP2: device pinhead:PINHD-2X20 -> pinhead:PINHD-1X6
- R1: value (none) -> 10K; device resistor:R-EU_R1206 -> rcl:R-US_M1206
- R2, R3, R4: value (none) -> 1K; device resistor:R-EU_R1206 -> rcl:R-US_M1206
- SV5: device con-lstb:MA08-1 -> pinhead:PINHD-1X8
- SV8: device con-lsta:FE08-1 -> pinhead:PINHD-1X8
- U1: value (none) -> STM32F103VCT6; device LP38690DT-3.3:LP38690DT-3.3 -> STM32F103VCT6:STM32F103VCT6
- X1: value 22-23-2021 -> 5566-4; device con-molex:22-23-2021 -> con-molex:5566-4
Connections:
- removed net 12V: C1.1, C4.1, C9.1, IC1.VI, IC2.VI, IC3.VI, R4.1, SV14.10, SV14.9, U$4.VOUT
- removed net 5V1: C5.1, IC2.VO, R1.1, X1-2.S
- removed net 5V_ESP: C10.1, IC3.VO, JP6.1, JP6.2
- removed net ESP_EN: JP2.24
- removed net ESP_REC: JP6.15, JP6.16
- removed net ESP_RX: JP1.26, JP5.23, JP5.24, S2.S, S2.S@1
- removed net ESP_TRANS: JP6.13, JP6.14
- removed net ESP_TX: JP1.28, JP5.25, JP5.26, S3.S, S3.S@1
- removed net FPGA_REC: JP2.26, R5.1
- removed net INPUT: U$5.S, U1.A, U1.~A, U2.A, U2.~A, U3.A, U3.~A
- removed net N$10: LED3.A, R3.2
- removed net N$11: JP5.11, JP5.12
- removed net N$12: JP5.13, JP5.14
- removed net N$13: LED4.A, R4.2
- removed net N$14: JP5.15, JP5.16
- removed net N$15: JP5.17, JP5.18
- removed net N$16: LED5.A, R5.2
- removed net N$17: JP5.19, JP5.20
- removed net N$18: JP5.21, JP5.22
- removed net N$23: JP5.27, JP5.28
- removed net N$24: JP5.29, JP5.30
- removed net N$27: JP6.5, JP6.6
- removed net N$28: JP6.7, JP6.8
- removed net N$29: JP6.10, JP6.9
- removed net N$30: JP6.11, JP6.12
- removed net N$38: JP6.27, JP6.28
- removed net N$39: JP6.29, JP6.30
- removed net N$41: JP6.25, JP6.26
- removed net N$6: JP5.5, JP5.6
- removed net N$8: JP5.7, JP5.8
- removed net N$9: JP5.10, JP5.9
- removed net SUPP: J5.+, U$5.P
- new net 5V_EXT: JP1.3
- new net 5V_REG: C13.1, IC2.IN_1, IC2.IN_2, IC3.G, IC3.VCC, IC4.G, IC4.VCC, J1.2, J2.5, J3.2, J4.5, J5.2, J6.5, J7.5, J8.2, JP1.2, MD1.5V, MD2.5V, MD3.5V, MD4.5V, MD5.5V, R2.2, SV8.5
- new net M1EAN: IC3.1A, J1.5
- new net M1EA_RECT: IC3.1Y
- new net M1EBN: IC3.2B, J1.7
- new net M1EB_RECT: IC3.2Y
- new net M2EAN: J3.5
- new net M2EA_RECT: IC3.4Y
- new net M2EBN: IC3.3B, J3.7
- new net M2EB_RECT: IC3.3Y
- new net M3EAN: IC3.4B, IC4.1A, J5.5
- new net M3EA_RECT: IC4.1Y
- new net M3EBN: IC4.2B, J5.7
- new net M3EB_RECT: IC4.2Y
- new net M4EAN: IC4.4B, J8.5
- new net M4EA_RECT: IC4.4Y
- new net M4EBN: IC4.3B, J8.7
- new net M4EB_RECT: IC4.3Y
- new net N$2: 3V3_LD.A, R3.1
- new net N$3: C11.1, IC1.VO, JP1.1
- new net NRF_CE: M1.CE
- new net NRF_CSN: M1.CSN, NRF_STATUS.C
- new net NRF_IRQ: M1.IRQ
- new net NRF_MISO: M1.MISO
- new net NRF_MOSI: M1.MOSI
- new net NRF_SCK: M1.SCK
- new net NRST: C10.1, JP2.5, S1.1, S1.2
- new net SWCLK: JP2.2, U1A.PA14
- new net SWDIO: JP2.4, U1A.PA13
- new net SWO: JP2.6, U1A.PB3
- net 18V: now also C12.1, IC1.VI, MD1.18V, MD2.18V, MD3.18V, MD4.18V, MD5.18V; no longer R3.1, SV1.10, SV1.9, SV2.10, SV2.9, SV3.10, SV3.9, SV4.10, SV4.9, U$4.VIN, U1.K, U2.K, U3.K
- net CHARGE: no longer JP2.16
- net DONE: no longer JP2.18
- net GND: now also 3V3_LD.C, 5V_LD.C, C11.2, C12.2, C13.2, C14.2, C15.2, C16.2, C2.2, C6.2, C7.2, C8.2, IC3.!G, IC4.!G, IC4.GND, J2.4, J4.4, J5.3, J8.3, JP2.3, M1.GND, MD1.GND, MD2.GND, MD3.GND, MD4.GND, MD5.GND, R1.1, S1.3, S1.4, U1C.VREF-, U1C.VSSA, U1C.VSS_1, U1C.VSS_2, U1C.VSS_3, U1C.VSS_4, U1C.VSS_5; no longer C2.1, C6.1, C7.1, C8.1, J2.3, J4.3, J5.-, J8.4, J9.4, JP1.1, JP1.19, JP1.20, JP1.39, JP2.2, JP2.40, JP5.3, JP5.4, JP6.3, JP6.4, LED1.C, LED2.C, LED3.C, LED4.C, LED5.C, S2.P, S2.P@1, S3.P, S3.P@1, SV1.1, SV1.2, SV14.1, SV14.2, SV2.1, SV2.2, SV3.1, SV3.2, SV4.1, SV4.2, U$4.GND, U$4.GNDO, X1-1.S
- net IR1: no longer JP2.25
- net IR2: no longer JP2.27
- net IR3: no longer JP2.15
- net KICK: no longer JP2.22
- net KICK_CHIP: no longer JP2.20
- net M11: now also MD1.M1; no longer SV6.6, SV6.7
- net M11A: now also MD1.M1A; no longer JP1.13, SV2.8
- net M11B: now also MD1.M1B; no longer JP1.11, SV2.7
- net M12: now also MD1.M2; no longer SV6.4, SV6.5
- net M12A: now also MD1.M2A; no longer JP1.9, SV2.6
- net M12B: now also MD1.M2B; no longer JP1.7, SV2.5
- net M13: now also MD1.M3; no longer SV6.2, SV6.3
- net M13A: now also MD1.M3A; no longer JP1.5, SV2.4
- net M13B: now also MD1.M3B; no longer JP1.3, SV2.3
- net M1ACS_OUT: now also MD1.ACS; no longer C2.2, JP6.17, JP6.18, SV6.8
- net M1EA: now also IC3.1B; no longer JP1.6
- net M1EB: now also IC3.2A; no longer JP1.4
- net M1H1: no longer JP1.8
- net M1H2: no longer JP1.10
- net M1H3: no longer JP1.12
- net M21: now also MD2.M1, X1-1.S; no longer SV7.6, SV7.7, X2-1.S
- net M21A: now also MD2.M1A; no longer JP1.27, SV1.8
- net M21B: now also MD2.M1B; no longer JP1.29, SV1.7
- net M22: now also MD2.M2, X1-2.S; no longer SV7.4, SV7.5, X2-2.S
- net M22A: now also MD2.M2A; no longer JP1.31, SV1.6
- net M22B: now also MD2.M2B; no longer JP1.33, SV1.5
- net M23: now also MD2.M3, X1-3.S; no longer SV7.2, SV7.3, X2-3.S
- net M23A: now also MD2.M3A; no longer JP1.35, SV1.4
- net M23B: now also MD2.M3B; no longer JP1.37, SV1.3
- net M2ACS_OUT: now also MD2.ACS; no longer C6.2, JP6.19, JP6.20, SV7.8
- net M2EA: no longer JP1.32
- net M2EB: now also IC3.3A; no longer JP1.30
- net M2H1: now also J2.1; no longer J7.1, JP1.34
- net M2H2: now also J2.2; no longer J7.2, JP1.36
- net M2H3: now also J2.3; no longer J7.3, JP1.38
- net M31: now also MD3.M1, X2-1.S; no longer SV13.6, SV13.7, X4-1.S
- net M31A: now also MD3.M1A; no longer JP2.4, SV3.8
- net M31B: now also MD3.M1B; no longer JP2.6, SV3.7
- net M32: now also MD3.M2, X2-2.S; no longer SV13.4, SV13.5, X4-2.S
- net M32A: now also MD3.M2A; no longer JP2.8, SV3.6
- net M32B: now also MD3.M2B; no longer JP2.10, SV3.5
- net M33: now also MD3.M3, X2-3.S; no longer SV13.2, SV13.3, X4-3.S
- net M33A: now also MD3.M3A; no longer JP2.12, SV3.4
- net M33B: now also MD3.M3B; no longer JP2.14, SV3.3
- net M3ACS_OUT: now also MD3.ACS; no longer C7.2, JP6.21, JP6.22, SV13.8
- net M3EA: now also IC3.4A, IC4.1B, J5.6; no longer J2.6, JP2.3
- net M3EB: now also IC4.2A, J5.8; no longer J2.8, JP2.5
- net M3H1: now also J4.1; no longer J8.1, JP2.7
- net M3H2: now also J4.2; no longer J8.2, JP2.9
- net M3H3: now also J4.3; no longer J8.3, JP2.11
- net M41: now also MD4.M1, X4-1.S; no longer SV18.6, SV18.7, X5-1.S
- net M41A: now also MD4.M1A; no longer JP2.38, SV4.8
- net M41B: now also MD4.M1B; no longer JP2.36, SV4.7
- net M42: now also MD4.M2, X4-2.S; no longer SV18.4, SV18.5, X5-2.S
- net M42A: now also MD4.M2A; no longer JP2.34, SV4.6
- net M42B: now also MD4.M2B; no longer JP2.32, SV4.5
- net M43: now also MD4.M3, X4-3.S; no longer SV18.2, SV18.3, X5-3.S
- net M43A: now also MD4.M3A; no longer JP2.30, SV4.4
- net M43B: now also MD4.M3B; no longer JP2.28, SV4.3
- net M4ACS_OUT: now also MD4.ACS; no longer C8.2, JP6.23, JP6.24, SV18.8
- net M4EA: now also IC4.4A, J8.6; no longer J4.6, JP2.31
- net M4EB: now also IC4.3A, J8.8; no longer J4.8, JP2.29
- net M4H1: now also J7.1; no longer J9.1, JP2.33
- net M4H2: now also J7.2; no longer J9.2, JP2.35
- net M4H3: now also J7.3; no longer J9.3, JP2.37
- net MD1: now also MD5.M1; no longer SV17.6, SV17.7
- net MD1A: now also MD5.M1A; no longer JP1.15, SV14.8
- net MD1B: now also MD5.M1B; no longer JP1.17, SV14.7
- net MD2: now also MD5.M2; no longer SV17.4, SV17.5
- net MD2A: now also MD5.M2A; no longer JP2.13, SV14.6
- net MD2B: now also MD5.M2B; no longer JP1.21, SV14.5
- net MD3: now also MD5.M3; no longer SV17.2, SV17.3
- net MD3A: now also MD5.M3A; no longer JP1.23, SV14.4
- net MD3B: now also MD5.M3B; no longer JP1.25, SV14.3
- net MDACS_OUT: now also MD5.ACS; no longer SV17.8
- net MDH1: no longer JP1.16
- net MDH2: no longer JP1.18
- net MDH3: no longer JP2.17
- net N$1: now also R1.2, U1A.BOOT0; no longer JP5.1, JP5.2
- net N$4: now also 5V_LD.A, R2.1; no longer LED1.A, R1.2
- net N$7: now also NRF_STATUS.A, R4.1; no longer LED2.A, R2.2
- net VCC: now also C1.1, C14.1, C15.1, C16.1, C2.1, C4.1, C5.1, C6.1, C7.1, C8.1, C9.1, IC2.OUT, JP2.1, M1.VCC, R3.2, R4.2, U1C.VBAT, U1C.VDDA, U1C.VDD_1, U1C.VDD_2, U1C.VDD_3, U1C.VDD_4, U1C.VDD_5, U1C.VREF+; no longer IC1.VO, J1.2, J2.2, J3.2, J4.2, J6.5, J7.5, J8.5, J9.5, R2.1, SV13.1, SV17.1, SV18.1, SV6.1, SV7.1, SV8.5
Other:
- note removed: "12V"
- note removed: "5V"
- note removed: "5V1"
- note removed: "Dribbler"
- note removed: "ESP32"
- note removed: "FPGA"
- note removed: "Input"
- note removed: "Kicker"
- note removed: "Power Supply"
- note removed: "Status LED"
- moved on the sheet: C1, C10, C2, C3, C4, C5, C6, C7, C8, C9, IC1, J1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
